File: kicad/arc/arc.kicad_sch (KiCad schematic)
At the start: 13 parts, among them J1 Conn_01x08, J2 Conn_01x03, J3 Conn_01x03, J4 Conn_01x03, J5 Conn_01x03, J6 Conn_01x03, J7 Conn_01x03, J8 Conn_01x03, J9 Conn_01x03, U1 ESP32-S3-WROOM-1U-N16R8, U2 BL5612, U3 TPS63020DSJR, U4 BL5612

Commit message: fixed it just a mare '#'
Parts:
- removed U3: TPS63020DSJR, Package_SON:Texas_S-PVSON-N14_ThermalPad, symbol TPS63020DSJR:TPS63020DSJR
Other:
- note added: "GND"
- note added: "L/R"
- note added: "SCK"
- note added: "SD"
- note added: "VDD"
- note added: "WS"

Commit message: fixed
Parts:
- added U3: TPS63020DSJR, DSJ14_2P85X1P58, symbol 2026-09-04_08-16-50:TPS63020DSJR
Connections:
- net at J7.1 (Pin_1): now also J3.1 (Pin_1), J5.1 (Pin_1), J9.1 (Pin_1), U1.13 (IO19)
- net at J7.2 (Pin_2): now also J3.2 (Pin_2), J5.2 (Pin_2), J9.2 (Pin_2), U1.14 (IO20)
- net at J7.3 (Pin_3): now also J1.7 (Pin_7), J2.2 (Pin_2), J4.2 (Pin_2), J5.3 (Pin_3), J6.2 (Pin_2), J8.2 (Pin_2), J9.3 (Pin_3), U1.2 (3V3)
- net at J6.1 (Pin_1): now also J8.1 (Pin_1), U1.11 (IO18)
- net at J6.3 (Pin_3): now also J2.3 (Pin_3), J3.3 (Pin_3), J4.3 (Pin_3), J8.3 (Pin_3)
- net at U1.12 (IO8): now also J2.1 (Pin_1), J4.1 (Pin_1)
- new net: U3.1 (VINA), U3.12 (EN)
- new net: U3.15 (EPAD), U3.2 (GND)

Commit message: devlog 2
Parts:
- added BZ1, BZ2: Buzzer, symbol Device:Buzzer
- added J10: oled, symbol Connector:Conn_01x04_Pin
- added L1: 1.5 uH, Inductor_SMD:L_0201_0603Metric_Pad0.64x0.40mm_HandSolder, symbol Device:L
- added R1: 560k, Resistor_SMD:R_01005_0402Metric, symbol Device:R
- added R2: 100k, symbol Device:R
- added ST1, blo1, blo2, mic1, mic2, mic3, mic4: 100 nf, symbol Device:C
- added ST2: 22 uf, symbol Device:C
- added ST3: 10 uf, symbol Device:C
- added m1: motor 1, symbol Connector_Generic:Conn_01x02
- added m2: motor, symbol Connector_Generic:Conn_01x02
- renumbered U4 to bl1, U2 to bl2
Connections:
- net at J1.7 (Pin_7), J2.2 (Pin_2), J4.2 (Pin_2)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: now also U3.4 (VOUT), U3.5 (VOUT), J10.1 (Pin_1), mic1.1, mic2.2, mic3.2
- net at J2.3 (Pin_3), J3.3 (Pin_3), J4.3 (Pin_3)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: now also J1.8 (Pin_8), U1.1 (GND), U3.13 (PS/SYNC), U3.15 (EPAD), U3.2 (GND), bl1.5 (GND), bl2.5 (GND), BZ1.2 (-), BZ2.2 (-), J10.2 (Pin_2), R2.1, ST1.2, ST2.1, ST3.1, mic1.2, mic3.1
- net at U1.19 (IO11): now also J10.3 (Pin_3)
- net at U1.20 (IO12): now also J10.4 (Pin_4)
- net at U1.28 (IO35): now also BZ2.1 (+)
- net at U1.29 (IO36): now also BZ1.1 (+)
- net at bl1.6 (OUTB): now also blo1.1, m1.2 (Pin_2)
- net at bl1.7 (OUTA): now also blo1.2, m1.1 (Pin_1)
- net at bl1.8 (VM), bl2.8 (VM): now also U3.1 (VINA), U3.10 (VIN), U3.11 (VIN), U3.12 (EN), R1.1, ST1.1, ST3.2
- net at bl2.6 (OUTB): now also blo2.1, m2.2 (Pin_2)
- net at bl2.7 (OUTA): now also blo2.2, m2.1 (Pin_1)
- net at U3.3 (FB): now also R1.2, R2.2
- net at U3.6 (L2): now also U3.7 (L2), L1.1
- net at U3.8 (L1): now also U3.9 (L1), L1.2
- net GND: no longer names the net of U1.40 (GND)
- no-connect marks 0 -> 14
